File: hardware/dongle-pro-power/dongle-pro-power.kicad_sch (KiCad schematic)
At the start: 153 parts, among them J1 TYPE-C 24P QT, J2 TYPE-C 24P QT, J3 TC2030-IDC-NL, J4 TYPE-C 24P QT, Q1 AOD4184A, Q2 AOD4184A, Q3 AOD4184A, Q4 AOD4184A, Q5 AOD4184A, SW1 TS-1187A-B-A-B, U1 RP2354A, U10 AP22653W6-7, U11 STUSB4500QTR, U12 LM74800QDRRRQ1, U13 LM74800QDRRRQ1, U14 TPS54331DR, U15 INA180A1IDBVR, U2 FUSB302BMPX, U3 HD3SS3220RNHR, U4 GL3510-OSY52, U5 RT9013-33GB, U6 TLV70212DBVR, U7 HD3SS3212IRKSR, U8 74AVC1T45GW,125, U9 74AVC1T45GW,125, Y1 X322512MSB4SI, Y2 25MHz

Commit message: undome
Parts:
- removed L3: 10uH, dongle-lite:IND-SMD_L2.0-W1.6_AOTA-B201610S3R3-101-T, symbol dongle-lite:AOTA-B201610S3R3-101-T
- removed Q1, Q2, Q3, Q4, Q5: AOD4184A, dongle-lite:TO-252-2_L6.6-W6.1-P4.57-LS9.9-TL-CW, symbol dongle-lite:AOD4184A
- removed R26: 10mR, dongle-lite:R0402, symbol dongle-lite:0402WGF1002TCE
- added C73, C74: 100nF, dongle-lite:C0402, symbol dongle-lite:CL05B104KO5NNNC
- added D23, D24: SMBJ24A, dongle-lite:SMB_L4.6-W3.6-LS5.3-RD, symbol dongle-lite:SMBJ24A-C87268
- added L3: 10uH, dongle-lite:IND-SMD_L5.0-W5.0-1, symbol dongle-lite:SLW5040S100MST
- added Q1, Q2, Q3, Q4, Q5: NVMFD5853NL-HXY, dongle-lite:PDFN-8_L5.8-W4.9-P1.27-LS6.1-BL, symbol dongle-lite:NVMFD5853NL
- added R26: 10mR-2512, dongle-lite:RES-SMD_L6.4-W3.2-R2512, symbol dongle-lite:HOJLR2512-3W-10MR-1%
- added R41, R42: 1k, dongle-lite:R0402, symbol dongle-lite:0402WGF1001TCE
Connections:
- net +5V_BUCK: now also L3.2; no longer C65.1, C65.2, U14.1 (BOOT), U14.8 (PH)
- net GND: now also U12.7 (GND), U13.7 (GND), C73.2, C74.2, D23.2 (A), D24.2 (A), Q5.1 (S), Q5.2 (S), Q5.3 (S); no longer U12.13 (RTN), U13.13 (RTN)
- net PWR_VBUS: now also D23.1 (C), Q1.1 (S), Q1.2 (S), Q1.3 (S), R41.1, R42.2; no longer U11.18 (VBUS_VS_DISCH), U11.9 (DISCH), U12.10 (VS), U12.3 (VSNS)
- net SRC20: now also Q2.1 (S), Q2.2 (S), Q2.3 (S), R26.1; no longer U12.12 (C)
- net SRC20_DG: now also Q1.4 (G)
- net TGT_VBUS: now also D24.1 (C), Q4.1 (S), Q4.2 (S), Q4.3 (S), R26.2; no longer U13.12 (C)
- net VBUS_DISCHG: now also Q5.4 (G)
- net VSAFE_DG: now also Q3.4 (G)
- net VSAFE_SRC: now also Q3.1 (S), Q3.2 (S), Q3.3 (S); no longer U13.10 (VS), U13.3 (VSNS)
- net at U13.8 (HGATE): now also Q4.4 (G)
- net at U12.8 (HGATE): now also Q2.4 (G)
- net at R35.2, R36.1, R36.2: now also Q5.5 (D), Q5.6 (D), Q5.7 (D), Q5.8 (D), Q5.9 (D)
- net SRC20_SW renamed SRC20_MID
- net SRC20_MID: now also U12.10 (VS), U12.12 (C), U12.3 (VSNS), C73.1, Q1.5 (D), Q1.6 (D), Q1.7 (D), Q1.8 (D), Q1.9 (D), Q2.5 (D), Q2.6 (D), Q2.7 (D), Q2.8 (D), Q2.9 (D)
- net VSAFE_SW renamed VSAFE_MID
- net VSAFE_MID: now also U13.10 (VS), U13.12 (C), U13.3 (VSNS), C74.1, Q3.5 (D), Q3.6 (D), Q3.7 (D), Q3.8 (D), Q3.9 (D), Q4.5 (D), Q4.6 (D), Q4.7 (D), Q4.8 (D), Q4.9 (D)
- new net: C65.1, U14.1 (BOOT)
- new net BUCK_PH: C65.2, L3.1, U14.8 (PH)
- new net STUSB_DIS: R42.1, U11.9 (DISCH)
- new net STUSB_VS: R41.2, U11.18 (VBUS_VS_DISCH)
