File: hardware/dongle-pro/dongle-pro.kicad_sch (KiCad schematic)
At the start: 111 parts, among them J1 TYPE-C 24P QT, J2 TYPE-C 24P QT, J3 TC2030-IDC-NL, SW1 TS-1187A-B-A-B, U1 RP2354A, U10 AP22653W6-7, U2 FUSB302BMPX, U3 HD3SS3220RNHR, U4 GL3510-OSY52, U5 RT9013-33GB, U6 TLV70212DBVR, U7 HD3SS3212IRKSR, U8 74AVC1T45GW,125, U9 74AVC1T45GW,125, Y1 X322512MSB4SI, Y2 25MHz

Commit message: TC2030 boot-switch wiring, LCSC part fixes, and a Dongle-Lite case (#12)
* Wire TC2030 pin 6 to the boot switch on both dongle boards

Pin 6 was unconnected. Tying it to BOOT_SW lets the SWD probe hold the
board in BOOTSEL without anyone reaching for SW1, which matters when the
running firmware can't be asked to reboot into the bootrom over USB.

* Correct two LCSC part numbers in the Dongle-Lite symbol library

The 330R 0402 resistor and the 4.7uF 0402 capacitor both carried codes
that don't resolve to those parts at JLCPCB.

* Add a 3D-printable case for the Dongle-Lite board

Two-piece CadQuery enclosure for dongle-lite-1s4l, driven off the board's
own dimensions. `uv run case.py` writes a STEP assembly plus print-ready
STLs for the tray and lid. Generated output stays out of git.
Parts:
- C6, C7, C9: LCSC C52923 -> C368809
- R12: LCSC C25905 -> C25105
Connections:
- net BOOT_SW: now reaches R13.2, SW1.1 (A), SW1.2 (B)
- net BOOT_SW: now also J3.6
- no-connect marks 63 -> 62
