File: hardware/dongle-lite/dongle-lite-1s4l.kicad_pcb (KiCad board)
At the start: 4 copper layers, 22 x 77 mm, 66 parts, among them J1 TYPE-C-31-M-12, J2 TYPE-C-31-M-12, J3 TC2030-IDC-NL, SW1 TS-1187A-B-A-B, U1 RP2354A, U10 AP22653W6-7, U2 FUSB302BMPX, U3 CH334F, U5 RT9013-33GB, U6 TLV70212DBVR, U8 74AVC1T45GW,125, U9 74AVC1T45GW,125, Y1 X322512MSB4SI, Y2 X322512MSB4SI

Commit message: Leave the hub's PSELF and RESET#/CDP pins open (#13)
Both pins are strap inputs sampled at power-up, and both were being driven to
the wrong state. Adafruit's CH334F breakout (product 5997) leaves each one
open; matching it fixes a bug that killed every restore through the dongle.

PSELF (18) was tied to GND, so the hub advertised bus-powered and its
downstream ports could only promise one unit load, 100 mA. Every Apple
restore-stage device asks for 500 mA:

  DFU          0x1227   unconfigured, but works -- DFU is endpoint-0 control
                        transfers only, which are legal in Address state
  Recovery     0x1281   configures
  MacBook Pro  0x12ac   kUSBFailedRequestedPower = 500, restore dies here

The last stage is the first that needs interfaces, and interfaces only exist
inside a configuration. Left open the pin floats high on its internal pull-up,
which is self-powered -- 500 mA per port, exactly the ask. The board still
draws from the host's VBUS; this is a declaration, not a supply, and nothing
draws the current either way (the target runs on its own battery and there is
no per-port VBUS switching).

RESET#/CDP (16) was held high by R5. That pin is also sampled at power-up:
high enables CDP, the downstream charging-port advertisement, and disables the
hub's low-power sleep. The datasheet wants it "completely suspended when not
reset". R5 is removed; the pin keeps its ~25k internal pull-up.

Fab package regenerated: 91 vias (was 93), 56 placements (was 57), 10k
quantity down to 2. DRC 0 violations, 0 unconnected.
Parts:
- removed R5: 10k, dongle-lite:R0402
Connections:
- U3 pad 16: HUB_RSTB -> unconnected-(U3-RESETCDP-Pad16)
- U3 pad 18: GND -> unconnected-(U3-PSELF-Pad18)
Routing:
- net HUB_RSTB: track 12.5 -> 0.00 mm, vias 2 -> 0
- net GND: track 285.9 -> 284.8 mm
- net HUB_3V3: track 16.8 -> 15.9 mm
