File: hardware/dongle-lite/dongle-lite.kicad_sch (KiCad schematic)
At the start: 54 parts, among them J1 TYPE-C-31-M-12, J2 TYPE-C-31-M-12, SW1 TS-1187A-B-A-B, U1 RP2040, U10 AP22653W6-7, U2 FUSB302BMPX, U3 CH334F, U4 W25Q32JVSSIQ, U5 RT9013-33GB, U6 TLV70212DBVR, U8 74AVC1T45GW,125, U9 74AVC1T45GW,125, Y1 X322512MSB4SI, Y2 X322512MSB4SI

Commit message: Add single-sided 4-layer dongle-lite variant and JLCPCB fab packages
- New dongle-lite-1s4l: single-sided 4-layer board for JLCPCB Economic
  PCBA (all parts on top), fully routed with 0 DRC errors
- Use uniform 0.45mm/0.20mm vias (JLCPCB standard 4-layer via, 0.125mm
  annular ring) so the board avoids the small-hole 4-wire Kelvin test
  upcharge
- Generate fab packages for both the 6-layer and single-sided variants:
  gerbers, Excellon drill, grouped BOM, CPL, and STEP models
- Add Tag-Connect TC2030 and test-point pad footprints
- Refresh passive/connector/QFN footprints, schematic, symbol, and the
  board-gen scripts
- Drop stale handoff/BOM/wiring notes now that the boards are finalized

- Ignore Freerouting .dsn/.ses round-trip intermediates
Parts:
- removed C6: 1uF, dongle-lite:C0402, symbol dongle-lite:CL05A105KA5NQNC
- removed C7, C9: 100nF, dongle-lite:C0402, symbol dongle-lite:CL05B104KO5NNNC
- removed U1: RP2040, dongle-lite:LQFN-56_L7.0-W7.0-P0.4-EP, symbol dongle-lite:RP2040
- removed U4: W25Q32JVSSIQ, dongle-lite:SOIC-8_L5.2-W5.2-P1.27-LS7.9-BL, symbol dongle-lite:W25Q32JVSSIQ_C2834491
- added C27: 100nF, dongle-lite:C0402, symbol dongle-lite:CL05B104KO5NNNC
- added C6, C7, C9: 4.7uF, dongle-lite:C0402, symbol dongle-lite:CL05A475KP5NRNC
- added J3: TC2030-IDC-NL, dongle-lite:Tag-Connect_TC2030-IDC-NL_2x03_P1.27mm_Vertical, symbol dongle-lite:TC2030
- added L1: 3.3uH, dongle-lite:IND-SMD_L2.0-W1.6_AOTA-B201610S3R3-101-T, symbol dongle-lite:AOTA-B201610S3R3-101-T
- added R12: 33, dongle-lite:R0402, symbol dongle-lite:0402WGF330JTCE
- added R13: 1k, dongle-lite:R0402, symbol dongle-lite:0402WGF1001TCE
- added TP1: +5V, dongle-lite:TestPoint_Pad_D1.0mm, symbol dongle-lite:TP
- added TP2: +3V3, dongle-lite:TestPoint_Pad_D1.0mm, symbol dongle-lite:TP
- added TP3: +1V2, dongle-lite:TestPoint_Pad_D1.0mm, symbol dongle-lite:TP
- added TP4: +1V1, dongle-lite:TestPoint_Pad_D1.0mm, symbol dongle-lite:TP
- added TP5: TGT_VBUS, dongle-lite:TestPoint_Pad_D1.0mm, symbol dongle-lite:TP
- added TP6: GND, dongle-lite:TestPoint_Pad_D1.0mm, symbol dongle-lite:TP
- added TP7: RUN, dongle-lite:TestPoint_Pad_D1.0mm, symbol dongle-lite:TP
- added TP8: FUSB_INT, dongle-lite:TestPoint_Pad_D1.0mm, symbol dongle-lite:TP
- added U1: RP2354A, dongle-lite:QFN-60_L7.0-W7.0-P0.40-TL-EP3.4, symbol dongle-lite:RP2354A_C41378174
Connections:
- net XIN is gone; now on net GND: C1.1, Y1.1 (OSC1)
- net +1V1: now also C7.1, L1.2, TP4.1, U1.23 (DVDD), U1.39 (DVDD), U1.50 (VREG_FB), U1.6 (DVDD)
- net +1V2: now also TP3.1
- net +3V3: now also C27.1, C6.1, J3.1, R12.1, TP2.1, U1.1 (IOVDD), U1.11 (IOVDD), U1.20 (IOVDD), U1.30 (IOVDD), U1.38 (IOVDD), U1.44 (ADC_AVDD), U1.45 (IOVDD), U1.49 (VREG_VIN), U1.53 (USB_OTP_VDD), U1.54 (QSPI_IOVDD)
- net +5V: now also TP1.1
- net FUSB_INT: now also TP8.1, U1.29 (GPIO18)
- net GND: now also C27.2, C6.2, C7.2, C9.2, J3.5, TP6.1, U1.21 (XIN), U1.47 (VREG_PGND), U1.61 (GND)
- net HUB_XI: now also C16.1; no longer C15.1
- net HUB_XO: now also C15.1; no longer C16.1
- net I2C_SCL: now also U1.28 (GPIO17)
- net I2C_SDA: now also U1.27 (GPIO16)
- net LED_STAT: now also U1.37 (GPIO25)
- net RUN: now also J3.3, TP7.1, U1.26 (RUN)
- net SBU1_DIR: now also U1.32 (GPIO20)
- net SBU1_UART: now also U1.34 (GPIO22)
- net SBU2_DIR: now also U1.33 (GPIO21)
- net SBU2_UART: now also U1.35 (GPIO23)
- net SHIFT_EN: now also U1.36 (GPIO24)
- net SWCLK: now also J3.4, U1.24 (SWCLK)
- net SWDIO: now also J3.2, U1.25 (SWDIO)
- net TGT_VBUS: now also TP5.1
- net TGT_VBUS_EN: now also U1.31 (GPIO19)
- net at SW1.1 (A), SW1.2 (B): now also R13.2
- net HOST_DM renamed HOST_D_N
- net HOST_DP renamed HOST_D_P
- net MCU_DM renamed MCU_D_N
- net MCU_D_N: now also U1.51 (USB_DM)
- net MCU_DP renamed MCU_D_P
- net MCU_D_P: now also U1.52 (USB_DP)
- net TGT_DM renamed TGT_D_N
- net TGT_DP renamed TGT_D_P
- net XOUT: no longer names the net of C2.1, Y1.3 (OSC2)
- net XOUT: now also U1.22 (XOUT)
- new net: C9.1, R12.2, U1.46 (VREG_AVDD)
- new net: R13.1, U1.60 (QSPI_SS)
- new net VREG_LX: L1.1, U1.48 (VREG_LX)
- no-connect marks 38 -> 44

Commit message: TC2030 boot-switch wiring, LCSC part fixes, and a Dongle-Lite case (#12)
* Wire TC2030 pin 6 to the boot switch on both dongle boards

Pin 6 was unconnected. Tying it to BOOT_SW lets the SWD probe hold the
board in BOOTSEL without anyone reaching for SW1, which matters when the
running firmware can't be asked to reboot into the bootrom over USB.

* Correct two LCSC part numbers in the Dongle-Lite symbol library

The 330R 0402 resistor and the 4.7uF 0402 capacitor both carried codes
that don't resolve to those parts at JLCPCB.

* Add a 3D-printable case for the Dongle-Lite board

Two-piece CadQuery enclosure for dongle-lite-1s4l, driven off the board's
own dimensions. `uv run case.py` writes a STEP assembly plus print-ready
STLs for the tray and lid. Generated output stays out of git.
Connections:
- net BOOT_SW: now reaches R13.2, SW1.1 (A), SW1.2 (B)
- net BOOT_SW: now also J3.6
- no-connect marks 44 -> 43

Commit message: Leave the hub's PSELF and RESET#/CDP pins open (#13)
Both pins are strap inputs sampled at power-up, and both were being driven to
the wrong state. Adafruit's CH334F breakout (product 5997) leaves each one
open; matching it fixes a bug that killed every restore through the dongle.

PSELF (18) was tied to GND, so the hub advertised bus-powered and its
downstream ports could only promise one unit load, 100 mA. Every Apple
restore-stage device asks for 500 mA:

  DFU          0x1227   unconfigured, but works -- DFU is endpoint-0 control
                        transfers only, which are legal in Address state
  Recovery     0x1281   configures
  MacBook Pro  0x12ac   kUSBFailedRequestedPower = 500, restore dies here

The last stage is the first that needs interfaces, and interfaces only exist
inside a configuration. Left open the pin floats high on its internal pull-up,
which is self-powered -- 500 mA per port, exactly the ask. The board still
draws from the host's VBUS; this is a declaration, not a supply, and nothing
draws the current either way (the target runs on its own battery and there is
no per-port VBUS switching).

RESET#/CDP (16) was held high by R5. That pin is also sampled at power-up:
high enables CDP, the downstream charging-port advertisement, and disables the
hub's low-power sleep. The datasheet wants it "completely suspended when not
reset". R5 is removed; the pin keeps its ~25k internal pull-up.

Fab package regenerated: 91 vias (was 93), 56 placements (was 57), 10k
quantity down to 2. DRC 0 violations, 0 unconnected.
Parts:
- removed R5: 10k, dongle-lite:R0402, symbol dongle-lite:0402WGF1002TCE
Connections:
- net GND: no longer U3.18 (PSELF)
- net HUB_RSTB: no longer names the net of U3.16 (~{RESET}/CDP)
- no-connect marks 43 -> 45
